Commit message: perfect

File: src/viola_gazebo/config/viola_gazebo.urdf.xacro (robot description, xacro)
@@ -5,4 +5,7 @@
         <parent link="world"/>
         <child link="base_link"/>
+        <origin
+        xyz="0 0 0.061927"
+        rpy="0 0 0" />
     </joint>
     <xacro:include filename="$(find viola_gazebo)/urdf/viola_gazebo.urdf" />

File: src/viola_gazebo/urdf/viola_gazebo.urdf (robot description, URDF)
Before this commit: robot viola_description, 9 links, 8 joints
Joints:
- joint joint1: limit lower=-2.27 upper=2.27 effort=100 velocity=1 -> lower=-2.27 upper=2.27 effort=1 velocity=1
- joint joint2: limit lower=-1.57 upper=1.57 effort=100 velocity=1 -> lower=-1.57 upper=1.57 effort=2.3 velocity=1
- joint joint3: limit lower=-1.57 upper=1.57 effort=100 velocity=1 -> lower=-1.57 upper=1.57 effort=2.3 velocity=1
- joint joint4: limit lower=-2.27 upper=2.27 effort=100 velocity=1 -> lower=-2.27 upper=2.27 effort=1 velocity=1
- joint joint5: limit lower=-1.57 upper=1.57 effort=100 velocity=1 -> lower=-1.57 upper=1.57 effort=1 velocity=1
- joint joint6: limit lower=-2.27 upper=2.27 effort=100 velocity=1 -> lower=-2.27 upper=2.27 effort=1 velocity=1
- joint joint7_left: limit lower=-0.03 upper=0 effort=5 velocity=3.14 -> lower=-0.03 upper=0 effort=1 velocity=3.14
- joint joint7_right: limit lower=-3.14 upper=3.14 effort=5 velocity=3.14 -> lower=-3.14 upper=3.14 effort=1 velocity=3.14
