Commit message: Update STL meshes and URDF files for cello and viola robots

File: src/cello_description/urdf/cello_description.urdf (robot description, URDF)
Before this commit: robot cello_description, 10 links, 9 joints
Links:
- link base_link: mass 0.860146103961966 -> 0.860146104031393
- link link1: mass 0.211492633912495 -> 0.211492634096808
- link link2: mass 0.227311190417969 -> 0.226428575789942
- link link4: mass 0.0850055961870255 -> 0.0831858188735885
- link link5: mass 0.0163654245254692 -> 0.0181852018389062
Joints:
- joint joint1: axis 0 0 -1 -> 0 0 1; origin xyz=0 0 0.0665 rpy=0 0 3.1416 -> xyz=0 0 0.0665 rpy=0 0 3.14159265358979
- joint joint2: origin xyz=0.0022 0 0.0638 rpy=-1.5708 -1.5708 0 -> xyz=0.0022 0 0.0638 rpy=1.5708 -1.5708 0
- joint joint3: origin xyz=0.2476 0.0396 0 rpy=0 0 1.5708 -> xyz=0.2476 -0.0396 0 rpy=0 0 -1.5708
- joint joint4: axis 0 0 -1 -> 0 0 1; origin xyz=0.26712 0.00308 0 rpy=-1.5708 0 -1.5708 -> xyz=0.26712 -0.00308 0 rpy=1.5708 0 1.5708
- joint joint5: origin xyz=0 0 0 rpy=1.5708 -1.5708 0 -> xyz=0 0 0 rpy=-1.5708 0 0
- joint joint6: origin xyz=0.17066 0.0048225 0 rpy=1.5708 0 1.5708 -> xyz=-0.001325 -0.17066 0 rpy=1.5708 -1.5708 0
- joint joint7_left: axis 0 0 1 -> 0 0 -1; limit lower=-0.03 upper=0 effort=5 velocity=3.14 -> lower=-3.14 upper=3.14 effort=5 velocity=3.14; origin xyz=0.01019 0 0 rpy=1.5708 0 3.1416 -> xyz=0 0.013687 0 rpy=1.5708 0 -1.5708
- joint joint7_right: axis 0 0 -1 -> 0 0 1; limit lower=-3.14 upper=3.14 effort=5 velocity=3.14 -> lower=-0.03 upper=0 effort=5 velocity=3.14; origin xyz=0.01019 0 0 rpy=1.5708 0 3.1416 -> xyz=0 0.013687 0 rpy=1.5708 0 -1.5708

File: src/viola_description/urdf/viola_description.urdf (robot description, URDF)
Before this commit: robot viola_description, 10 links, 9 joints
Links:
- link base_link: mass 0.34245 -> 0.342452235959815
- link link6: mass 0.0604810188118188 -> 0.0525962732183853
Joints:
- joint joint1: axis 7.6046E-05 0 -1 -> 7.60456271565632E-05 0 -0.999999997108531; origin xyz=0 -0.00968 0.0037502 rpy=0 0 -1.5708 -> xyz=0 -0.00968 0.00375020271826967 rpy=0 0 -1.5707963267949
- joint joint2: axis 0 0 -1 -> 0 0 -0.999999999999946; origin xyz=0.00081639 0 0.017894 rpy=1.5708 -1.5708 0 -> xyz=0.000816389136979258 0 0.0178942036719373 rpy=1.57079665385624 -1.5707963267949 0
- joint joint3: origin xyz=0.1622 -0.042677 0 rpy=0 0 -1.5708 -> xyz=0.162199430665324 -0.0426767500837757 0 rpy=0 0 -1.5707963267949
- joint joint4: origin xyz=0.13611 -0.001325 0 rpy=1.5708 0 1.5708 -> xyz=0.136105 -0.00132499999999894 0 rpy=1.5707963267949 0 1.5707963267949
- joint joint6: axis 0 1 0 -> 0 0 -1; origin xyz=-0.0048225 -0.17065 0 rpy=3.1416 0 3.1416 -> xyz=-0.0048225 -0.17065 0 rpy=1.5708 -1.5708 0
- joint joint7_left: origin xyz=0.01009 0 0 rpy=0 0 3.1416 -> xyz=0 0.0100900000000006 0 rpy=1.5707963267949 0 -1.5707963267949
- joint joint7_right: origin xyz=0.0100900000000006 0 0 rpy=0 0 3.14159265358979 -> xyz=0 0.0100900000000006 0 rpy=1.5707963267949 0 -1.5707963267949

File: src/viola_gazebo/urdf/viola_gazebo.urdf (robot description, URDF)
Before this commit: robot viola_description, 9 links, 8 joints
Links:
- link base_link: mass 0.34245 -> 0.342452235959815
- link link6: mass 0.0604810188118188 -> 0.0525962732183853
Joints:
- joint joint1: axis 7.6046E-05 0 -1 -> 7.60456271565632E-05 0 -0.999999997108531; origin xyz=0 -0.00968 0.0037502 rpy=0 0 -1.5708 -> xyz=0 -0.00968 0.00375020271826967 rpy=0 0 -1.5707963267949
- joint joint2: axis 0 0 -1 -> 0 0 -0.999999999999946; origin xyz=0.00081639 0 0.017894 rpy=1.5708 -1.5708 0 -> xyz=0.000816389136979258 0 0.0178942036719373 rpy=1.57079665385624 -1.5707963267949 0
- joint joint3: origin xyz=0.1622 -0.042677 0 rpy=0 0 -1.5708 -> xyz=0.162199430665324 -0.0426767500837757 0 rpy=0 0 -1.5707963267949
- joint joint4: origin xyz=0.13611 -0.001325 0 rpy=1.5708 0 1.5708 -> xyz=0.136105 -0.00132499999999894 0 rpy=1.5707963267949 0 1.5707963267949
- joint joint6: axis 0 1 0 -> 0 0 -1; origin xyz=-0.0048225 -0.17065 0 rpy=3.1416 0 3.1416 -> xyz=-0.0048225 -0.17065 0 rpy=1.5708 -1.5708 0
- joint joint7_left: origin xyz=0.01009 0 0 rpy=0 0 3.1416 -> xyz=0 0.0100900000000006 0 rpy=1.5707963267949 0 -1.5707963267949
- joint joint7_right: origin xyz=0.0100900000000006 0 0 rpy=0 0 3.14159265358979 -> xyz=0 0.0100900000000006 0 rpy=1.5707963267949 0 -1.5707963267949

Commit message: Update cello robot URDF and meshes, reorganize README sections

File: src/cello_description/urdf/cello_description.urdf (robot description, URDF)
Before this commit: robot cello_description, 10 links, 9 joints
Joints:
- joint joint1: axis 0 0 1 -> 0 0 -1
- joint joint2: axis 0 0 1 -> 0 0 -1
- joint joint3: axis 0 0 1 -> 0 0 -1
- joint joint4: axis 0 0 1 -> 0 0 -1
- joint joint5: axis 0 0 1 -> 0 0 -1
- joint joint7_left: axis 0 0 -1 -> 0 0 1
- joint joint7_right: axis 0 0 1 -> 0 0 -1

File: src/cello_gazebo/urdf/cello_gazebo.urdf (robot description, URDF)
Before this commit: robot cello_description, 9 links, 8 joints
Links:
- link base_link: mass 0.860146103961966 -> 0.860146104031393
- link link1: mass 0.211492633912495 -> 0.211492634096808
- link link2: mass 0.227311190417969 -> 0.226428575789942
- link link4: mass 0.0850055961870255 -> 0.0831858188735885
- link link5: mass 0.0163654245254692 -> 0.0181852018389062
Joints:
- joint joint1: origin xyz=0 0 0.0665 rpy=0 0 3.1416 -> xyz=0 0 0.0665 rpy=0 0 3.14159265358979
- joint joint2: axis 0 0 1 -> 0 0 -1; origin xyz=0.0022 0 0.0638 rpy=-1.5708 -1.5708 0 -> xyz=0.0022 0 0.0638 rpy=1.5708 -1.5708 0
- joint joint3: axis 0 0 1 -> 0 0 -1; origin xyz=0.2476 0.0396 0 rpy=0 0 1.5708 -> xyz=0.2476 -0.0396 0 rpy=0 0 -1.5708
- joint joint4: origin xyz=0.26712 0.00308 0 rpy=-1.5708 0 -1.5708 -> xyz=0.26712 -0.00308 0 rpy=1.5708 0 1.5708
- joint joint5: axis 0 0 1 -> 0 0 -1; origin xyz=0 0 0 rpy=1.5708 -1.5708 0 -> xyz=0 0 0 rpy=-1.5708 0 0
- joint joint6: origin xyz=0.17066 0.0048225 0 rpy=1.5708 0 1.5708 -> xyz=-0.001325 -0.17066 0 rpy=1.5708 -1.5708 0
- joint joint7_left: origin xyz=0.01019 0 0 rpy=1.5708 0 3.1416 -> xyz=0 0.013687 0 rpy=1.5708 0 -1.5708
- joint joint7_right: origin xyz=0.01019 0 0 rpy=1.5708 0 3.1416 -> xyz=0 0.013687 0 rpy=1.5708 0 -1.5708

Commit message: Update cello robot URDF parameters and meshes, adjust joint limits and orientation tolerance

File: src/cello_description/urdf/cello_description.urdf (robot description, URDF)
Before this commit: robot cello_description, 10 links, 9 joints
Links:
- link base_link: mass 0.860146104031393 -> 0.860146104012974
- link link1: mass 0.211492634096808 -> 0.21149263410611
- link link2: mass 0.226428575789942 -> 0.226428575799244
Joints:
- joint joint1: origin xyz=0 0 0.0665 rpy=0 0 3.14159265358979 -> xyz=0 0 0.0635 rpy=0 0 0
- joint joint2: origin xyz=0.0022 0 0.0638 rpy=1.5708 -1.5708 0 -> xyz=0.00220000000000002 0 0.0638 rpy=1.5707963267949 -1.5707963267949 0
- joint joint4: origin xyz=0.26712 -0.00308 0 rpy=1.5708 0 1.5708 -> xyz=0.267124999999999 -0.00308000000000425 0 rpy=1.5707963267949 0 1.5707963267949
- joint joint5: origin xyz=0 0 0 rpy=-1.5708 0 0 -> xyz=0 0 0 rpy=-1.5707963267949 0 0
- joint joint6: origin xyz=-0.001325 -0.17066 0 rpy=1.5708 -1.5708 0 -> xyz=-0.00132500000000002 -0.170658355416465 0 rpy=1.5707963267949 -1.5707963267949 0
- joint joint7_left: limit lower=-3.14 upper=3.14 effort=5 velocity=3.14 -> lower=-0.025 upper=0 effort=5 velocity=3.14; origin xyz=0 0.013687 0 rpy=1.5708 0 -1.5708 -> xyz=0 0.0136874999999999 0 rpy=1.5707963267949 0 -1.5707963267949
- joint joint7_right: limit lower=-0.03 upper=0 effort=5 velocity=3.14 -> lower=-0.025 upper=0 effort=5 velocity=3.14; origin xyz=0 0.013687 0 rpy=1.5708 0 -1.5708 -> xyz=0 0.0136874999999999 0 rpy=1.5707963267949 0 -1.5707963267949
