Commit message: update urdf

File: src/viola_description/urdf/viola_description.urdf (robot description, URDF)
Before this commit: robot viola_description, 10 links, 9 joints
Joints:
- joint joint1: axis 7.60456271565632E-05 0 -0.999999997108531 -> 7.60456271565632E-05 0 0.999999997108531; origin xyz=0 -0.00968 0.00375020271826967 rpy=0 0 -1.5707963267949 -> xyz=0 0 0.0657499999998377 rpy=0 0 0
- joint joint5: origin xyz=0 0 0 rpy=-1.5708 0 0 -> xyz=0 0 0 rpy=-1.57079632686333 0 0
- joint joint6: origin xyz=-0.0048225 -0.17065 0 rpy=1.5708 -1.5708 0 -> xyz=-0.00482250000000067 -0.170649999999999 0 rpy=1.5707963267949 -1.5707963267949 0

File: src/viola_gazebo/config/viola_gazebo.urdf.xacro (robot description, xacro)
@@ -6,5 +6,5 @@
         <child link="base_link"/>
         <origin
-        xyz="0 0 0.061927"
+        xyz="0 0 0.0"
         rpy="0 0 0" />
     </joint>

File: src/viola_gazebo/urdf/viola_gazebo.urdf (robot description, URDF)
Before this commit: robot viola_description, 9 links, 8 joints
Joints:
- joint joint1: axis 7.60456271565632E-05 0 -0.999999997108531 -> 7.60456271565632E-05 0 0.999999997108531; origin xyz=0 -0.00968 0.00375020271826967 rpy=0 0 -1.5707963267949 -> xyz=0 0 0.0657499999998377 rpy=0 0 0
- joint joint5: origin xyz=0 0 0 rpy=-1.5708 0 0 -> xyz=0 0 0 rpy=-1.57079632686333 0 0
- joint joint6: origin xyz=-0.0048225 -0.17065 0 rpy=1.5708 -1.5708 0 -> xyz=-0.00482250000000067 -0.170649999999999 0 rpy=1.5707963267949 -1.5707963267949 0

Commit message: 更新viola机器人URDF和运动参数，调整关节轴方向和运动轨迹

File: src/viola_description/urdf/viola_description.urdf (robot description, URDF)
Before this commit: robot viola_description, 10 links, 9 joints
Joints:
- joint joint1: axis 7.60456271565632E-05 0 0.999999997108531 -> 7.60456271565632E-05 0 -0.999999997108531

File: src/viola_gazebo/urdf/viola_gazebo.urdf (robot description, URDF)
Before this commit: robot viola_description, 9 links, 8 joints
Joints:
- joint joint1: axis 7.60456271565632E-05 0 0.999999997108531 -> 7.60456271565632E-05 0 -0.999999997108531
